File: circuit/Ac Temp Control .kicad_pcb (KiCad board)
At the start: 2 copper layers, 40 x 90 mm, 21 parts, among them J1 USB_B_Micro, Q1 P2N2222A, SW1 SW_Push, SW2 SW_Push, SW3 SW_Push, SW4 SW_Push, U1 AMS1117-5.0, U2 ATmega328-P, U3 DHT11, U4 TSOP382xx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

Commit message: Add files via upload
Parts:
- added D2: LED, LED_THT:LED_D1.8mm_W1.8mm_H2.4mm_Horizontal_O1.27mm_Z1.6mm, F.Cu at (193.0, 68.6)
- added J1: Conn_01x02_Male, Connector_Molex:Molex_KK-254_AE-6410-02A_1x02_P2.54mm_Vertical, F.Cu at (193.6, 62.9)
- added J2: Conn_01x05_Male, Connector_Molex:Molex_KK-254_AE-6410-05A_1x05_P2.54mm_Vertical, F.Cu at (181.8, 55.0)
- added R3: 100, Resistor_THT:R_Axial_DIN0207_L6.3mm_D2.5mm_P10.16mm_Horizontal, F.Cu at (165.2, 62.6)
- added R4: 4.7k, Resistor_THT:R_Axial_DIN0309_L9.0mm_D3.2mm_P12.70mm_Horizontal, F.Cu at (165.2, 53.5)
- added R5: 4.7k, Resistor_THT:R_Axial_DIN0309_L9.0mm_D3.2mm_P12.70mm_Horizontal, F.Cu at (165.2, 58.2)
- added SW1: SW_Push, Button_Switch_THT:SW_PUSH_6mm, F.Cu at (165.7, 66.7)
- added U1: CAT24C256, Package_DIP:DIP-8_W7.62mm_Socket, F.Cu at (181.6, 61.1)
- added VR1: L7805, Connector_Molex:Molex_KK-254_AE-6410-03A_1x03_P2.54mm_Vertical, F.Cu at (196.6, 55.0)
Connections:
- C1 pad 1: Net-(C1-Pad1) -> Net-(U2-Pad9)
- C1 pad 2: Net-(C1-Pad2) -> GND
- C2 pad 1: Net-(C2-Pad1) -> Net-(U2-Pad10)
- C2 pad 2: Net-(C2-Pad2) -> GND
- DISPLAY1 pad 3: Net-(DISPLAY1-Pad3) -> Net-(U2-Pad28)
- R1 pad 1: Net-(R1-Pad1) -> Net-(U2-Pad3)
- U2 pad 10: Net-(C2-Pad1) -> Net-(U2-Pad10)
- U2 pad 11: Net-(R4-Pad1) -> Net-(U2-Pad11)
- U2 pad 12: Net-(R5-Pad1) -> unconnected-(U2-Pad12)
- U2 pad 13: Net-(R6-Pad1) -> unconnected-(U2-Pad13)
- U2 pad 19: unconnected-(U2-Pad19) -> Net-(U2-Pad19)
- U2 pad 2: unconnected-(U2-Pad2) -> Net-(U2-Pad2)
- U2 pad 23: Net-(U2-Pad23) -> unconnected-(U2-Pad23)
- U2 pad 25: Net-(DISPLAY1-Pad3) -> unconnected-(U2-Pad25)
- U2 pad 28: unconnected-(U2-Pad28) -> Net-(U2-Pad28)
- U2 pad 3: unconnected-(U2-Pad3) -> Net-(U2-Pad3)
- U2 pad 4: Net-(R1-Pad1) -> Net-(U2-Pad4)
- U2 pad 5: Net-(U2-Pad5) -> Net-(J2-Pad3)
- U2 pad 6: Net-(R3-Pad1) -> Net-(U2-Pad6)
- U2 pad 9: Net-(C1-Pad1) -> Net-(U2-Pad9)
- U3 pad 2: Net-(U2-Pad23) -> Net-(U2-Pad2)
- U4 pad 1: Net-(U2-Pad5) -> Net-(U2-Pad4)
- Y1 pad 1: Net-(C1-Pad2) -> Net-(U2-Pad9)
- Y1 pad 2: Net-(C2-Pad2) -> Net-(U2-Pad10)
Routing:
- net Net-(R5-Pad1): track 0.00 -> 62.1 mm
- net Net-(R4-Pad1): track 62.1 -> 0.00 mm
- net Net-(U2-Pad23): track 16.5 -> 0.00 mm
- net Net-(U2-Pad2): track 0.00 -> 16.5 mm
- net GND: track 61.1 -> 69.7 mm
- net Net-(C1-Pad2): track 4.40 -> 0.00 mm
- net Net-(U2-Pad10): track 0.00 -> 4.36 mm
- net Net-(C2-Pad1): track 4.36 -> 0.00 mm
- net Net-(C2-Pad2): track 4.22 -> 0.00 mm
- net Net-(U2-Pad9): track 0.00 -> 3.20 mm
- net Net-(C1-Pad1): track 3.20 -> 0.00 mm

Commit message: PCB design and Gerber file generation
Parts:
- removed the J1 at (111.8, 43.2)
- removed the R3 at (133.4, 107.5)
- removed the R4 at (165.2, 53.5)
- removed the R5 at (165.2, 58.2)
- removed R6: 100, Resistor_THT:R_Axial_DIN0204_L3.6mm_D1.6mm_P5.08mm_Horizontal
- removed the SW1 at (131.7, 114.4)
- removed SW2, SW3, SW4: SW_Push, Button_Switch_THT:SW_PUSH_6mm
- removed the U1 at (110.5, 51.9)
- D1: value IR_EMITTER -> LED; footprint LED_THT:LED_D3.0mm_Horizontal_O1.27mm_Z2.0mm_IRGrey -> LED_THT:LED_D5.0mm
- D2: value LED -> IR_EMITTER; footprint LED_THT:LED_D1.8mm_W1.8mm_H2.4mm_Horizontal_O1.27mm_Z1.6mm -> LED_THT:LED_D5.0mm
- DISPLAY1: footprint SSD1306:128x64OLED -> Connector_Molex:Molex_KK-254_AE-6410-04A_1x04_P2.54mm_Vertical
- R1, R2: footprint Resistor_THT:R_Axial_DIN0204_L3.6mm_D1.6mm_P5.08mm_Horizontal -> Resistor_THT:R_Axial_DIN0207_L6.3mm_D2.5mm_P10.16mm_Horizontal
- R4, R5: value 100 -> 4.7k; footprint Resistor_THT:R_Axial_DIN0204_L3.6mm_D1.6mm_P5.08mm_Horizontal -> Resistor_THT:R_Axial_DIN0207_L6.3mm_D2.5mm_P10.16mm_Horizontal
- U1: value CAT24C256 -> ATmega328-P; footprint Package_DIP:DIP-8_W7.62mm_Socket -> Package_DIP:DIP-28_W7.62mm_Socket_LongPads
- U2: value ATmega328-P -> DHT11; footprint Package_DIP:DIP-28_W7.62mm_Socket_LongPads -> Sensor:Aosong_DHT11_5.5x12.0_P2.54mm
- U3: value DHT11 -> TSOP382xx; footprint Sensor:Aosong_DHT11_5.5x12.0_P2.54mm -> OptoDevice:Vishay_MINICAST-3Pin
- U4: value TSOP382xx -> CAT24C256; footprint OptoDevice:Vishay_MINICAST-3Pin -> Package_DIP:DIP-8_W7.62mm_Socket
- moved J1 83.7 mm to (119.3, 101.5), turned to 90 degrees
- moved VR1 83.3 mm to (123.4, 95.0), turned to 90 degrees
- moved D1 75.1 mm to (167.6, 107.4)
- moved U4 71.1 mm to (131.2, 112.8)
- moved R2 69.1 mm to (171.8, 100.9)
- moved D2 62.7 mm to (147.5, 111.7), turned to 180 degrees
- moved Q1 59.2 mm to (139.0, 104.5), turned to 90 degrees
- moved J2 48.5 mm to (166.7, 101.1), turned to 90 degrees
- moved U2 43.4 mm to (140.0, 118.5)
- moved SW1 39.6 mm to (129.1, 81.8)
- moved U1 38.6 mm to (153.8, 87.9)
- moved R1 38.5 mm to (146.6, 90.9), turned to -90 degrees
- moved C2 38.5 mm to (156.9, 124.7), turned to 180 degrees
- moved R4 34.6 mm to (141.3, 92.9), turned to 180 degrees
- moved C1 33.2 mm to (144.1, 124.7), turned to 0 degrees
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Connections:
- C1 pad 1: Net-(U2-Pad9) -> Net-(C1-Pad1)
- C2 pad 1: Net-(U2-Pad10) -> Net-(C2-Pad1)
- D1 pad 1: (no net) -> Net-(D1-Pad1)
- D1 pad 2: (no net) -> Net-(D1-Pad2)
- D2 pad 1: Net-(R3-Pad1) -> Net-(D2-PadA)
- D2 pad 2: Net-(D1-PadC) -> Net-(D1-Pad2)
- DISPLAY1 pad 2: Net-(D1-PadC) -> Net-(D1-Pad2)
- DISPLAY1 pad 3: Net-(U2-Pad28) -> Net-(DISPLAY1-Pad3)
- J2 pad 1: Net-(U2-Pad11) -> Net-(J2-Pad1)
- J2 pad 2: Net-(U2-Pad6) -> Net-(J2-Pad2)
- J2 pad 4: Net-(D1-PadC) -> Net-(D1-Pad2)
- Q1 pad 1: Net-(D1-PadA) -> Net-(D2-PadA)
- R1 pad 1: Net-(U2-Pad3) -> Net-(R1-Pad1)
- R2 pad 1: Net-(U2-Pad1) -> Net-(D1-Pad1)
- R2 pad 2: Net-(D1-PadC) -> Net-(R2-Pad2)
- R3 pad 2: Net-(U2-Pad19) -> Net-(D1-Pad2)
- R4 pad 1: Net-(R4-Pad1) -> Net-(DISPLAY1-Pad4)
- R4 pad 2: GND -> Net-(D1-Pad2)
- R5 pad 1: Net-(R5-Pad1) -> Net-(DISPLAY1-Pad3)
- R5 pad 2: GND -> Net-(D1-Pad2)
- SW1 pad 2: Net-(U2-Pad1) -> Net-(R3-Pad1)
- U1 pad 1: GND -> Net-(R3-Pad1)
- U1 pad 2: GND -> Net-(U1-Pad2)
- U1 pad 3: Net-(D1-PadC) -> Net-(R1-Pad1)
- U1 pad 4: GND -> Net-(U1-Pad4)
- U1 pad 5: Net-(DISPLAY1-Pad4) -> Net-(J2-Pad3)
- U1 pad 6: Net-(U2-Pad28) -> Net-(J2-Pad2)
- U1 pad 7: GND -> Net-(D1-Pad2)
- U1 pad 8: Net-(D1-PadC) -> GND
- U2 pad 1: Net-(U2-Pad1) -> Net-(D1-Pad2)
- U2 pad 2: Net-(U2-Pad2) -> Net-(U1-Pad2)
- U2 pad 3: Net-(U2-Pad3) -> unconnected-(U2-Pad3)
- U2 pad 4: Net-(U2-Pad4) -> GND
- U3 pad 1: Net-(D1-PadC) -> Net-(U1-Pad4)
- U3 pad 2: Net-(U2-Pad2) -> GND
- U3 pad 3: unconnected-(U3-Pad3) -> Net-(D1-Pad2)
- U4 pad 1: Net-(U2-Pad4) -> GND
- U4 pad 3: Net-(D1-PadC) -> Net-(D1-Pad2)
- VR1 pad 3: Net-(D1-PadC) -> Net-(D1-Pad2)
- Y1 pad 1: Net-(U2-Pad9) -> Net-(C1-Pad1)
- Y1 pad 2: Net-(U2-Pad10) -> Net-(C2-Pad1)
Routing:
- net Net-(D1-Pad2): track 0.00 -> 189.5 mm
- net GND: track 69.7 -> 239.7 mm
- net Net-(D1-PadC): track 120.8 -> 0.00 mm
- net Net-(DISPLAY1-Pad3): track 0.00 -> 105.3 mm
- net Net-(DISPLAY1-Pad4): track 0.00 -> 70.7 mm
- net Net-(R5-Pad1): track 62.1 -> 0.00 mm
- net Net-(U1-Pad2): track 0.00 -> 35.7 mm
- net Net-(R3-Pad1): track 0.00 -> 32.0 mm
- net Net-(C2-Pad1): track 0.00 -> 29.1 mm
- net Net-(D2-PadA): track 0.00 -> 27.8 mm
- net Net-(C1-Pad1): track 0.00 -> 27.7 mm
- net Net-(U1-Pad4): track 0.00 -> 23.4 mm
- net Net-(J2-Pad1): track 0.00 -> 21.7 mm
- net Net-(J2-Pad3): track 0.00 -> 16.6 mm
- net Net-(U2-Pad2): track 16.5 -> 0.00 mm
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Other:
- board size 40 x 90 mm -> 74.9 x 69.8 mm
